Commit message: .

File: robot_description/urdf/robot.urdf (robot description, URDF)
Before this commit: robot GeneratedRobot, 5 links, 4 joints
Links:
- link cube3: geometry collision box size=0.32 0.24 1.05; visual box size=0.32 0.24 1.05
Joints:
- joint base_link_to_intermediate2: origin xyz=-0.41295728577975466 -0.0005718776701223449 0.5 rpy=0 0 0 -> xyz=-0.4004037835261366 -0.0014640307123229834 0.5 rpy=0 0 0

Commit message: tt

File: robot_description/urdf/robot.urdf (robot description, URDF)
Before this commit: robot GeneratedRobot, 5 links, 4 joints
Links:
- removed link intermediate_link1
- removed link intermediate_link2
- added link arm1, mass 0.1; collision box size=0.05 0.05 0.5; visual box size=0.05 0.05 0.5
- added link arm2, mass 0.1; collision box size=0.05 0.05 0.5; visual box size=0.05 0.05 0.5
- link base_link: mass 1 -> 10
- link cube2: mass 1 -> 10
- link cube3: mass 1 -> 10
Joints:
- removed joint base_link_to_intermediate1
- removed joint base_link_to_intermediate2
- removed joint intermediate1_to_cube2
- removed joint intermediate2_to_cube3
- added joint arm1_to_cube2: type revolute, parent arm1, child cube2, origin xyz=0.185 0 0 rpy=0 0 0, axis 1 0 0, limit lower=-1.57 upper=1.57 effort=10.0 velocity=10
- added joint arm2_to_cube3: type revolute, parent arm2, child cube3, origin xyz=-0.185 0 0 rpy=0 0 0, axis 1 0 0, limit lower=-1.57 upper=1.57 effort=10.0 velocity=10
- added joint base_link_to_arm1: type prismatic, parent base_link, child arm1, origin xyz=0.234 0 0.5 rpy=0 0 0, axis 0 0 1, limit lower=0.0 upper=0.5 effort=1000.0 velocity=0.5
- added joint base_link_to_arm2: type prismatic, parent base_link, child arm2, origin xyz=-0.234 0 0.5 rpy=0 0 0, axis 0 0 1, limit lower=0.0 upper=0.5 effort=1000.0 velocity=0.5
