Commit message: feat: Add ROS2 Humble + MicroROS digital twin support
- Gazebo Ignition simulation with ros2_control
- ESP32 MicroROS controller for real hardware
- Movement scripts and test files
- Comprehensive README with project roadmap

File: tars_robot_description/urdf/tars_robot.xacro (robot description, xacro)
@@ -1,159 +1,143 @@
 <?xml version="1.0" ?>
 <robot name="tars_robot" xmlns:xacro="http://www.ros.org/wiki/xacro">
-<xacro:include filename="$(find tars_robot_description)/urdf/materials.xacro" />
-<xacro:include filename="$(find tars_robot_description)/urdf/tars_robot.trans" />
-<xacro:include filename="$(find tars_robot_description)/urdf/tars_robot.gazebo" />
-<link name="base_link">
-  <inertial>
-    <origin xyz="0.008319588931624738 -0.010813885260023571 0.14310917214526914" rpy="0 0 0"/>
-    <mass value="4.0824"/>
-    <inertia ixx="0.036398" iyy="0.039022" izz="0.005861" ixy="-0.0" iyz="-0.0" ixz="0.0"/>
-  </inertial>
-  <visual>
+  <xacro:include filename="$(find tars_robot_description)/urdf/materials.xacro" />
+  <xacro:include filename="$(find tars_robot_description)/urdf/tars_robot.trans" />
+  <xacro:include filename="$(find tars_robot_description)/urdf/tars_robot.gazebo" />
+  <!-- Dimensions (in meters) -->
+  <xacro:property name="leg_width" value="0.065"/>
+  <xacro:property name="leg_depth" value="0.065"/>
+  <xacro:property name="leg_height" value="0.255"/>
+  <xacro:property name="center_width" value="0.11"/> <!-- Y -->
+  <xacro:property name="center_depth" value="0.065"/> <!-- X -->
+  <xacro:property name="center_height" value="0.255"/> <!-- Z -->
+  <xacro:property name="gap" value="0.005"/> <!-- Gap between legs and center -->
+  <link name="dummy_link"></link>
+  <joint name="dummy_joint" type="fixed">
+    <parent link="dummy_link"/>
+    <child link="base_link"/>
+  </joint>
+  <!-- IMU Link -->
+  <link name="imu_link">
+    <inertial>
+      <mass value="0.01"/>
+      <inertia ixx="0.0001" ixy="0" ixz="0" iyy="0.0001" iyz="0" izz="0.0001"/>
+    </inertial>
+  </link>
+  <joint name="imu_joint" type="fixed">
+    <parent link="base_link"/>
+    <child link="imu_link"/>
     <origin xyz="0 0 0" rpy="0 0 0"/>
-    <geometry>
-      <mesh filename="file://$(find tars_robot_description)/meshes/base_link.stl" scale="0.001 0.001 0.001"/>
-    </geometry>
-    <material name="silver"/>
-  </visual>
-  <collision>
-    <origin xyz="0 0 0" rpy="0 0 0"/>
-    <geometry>
-      <mesh filename="file://$(find tars_robot_description)/meshes/base_link.stl" scale="0.001 0.001 0.001"/>
-    </geometry>
-  </collision>
-</link>
-<link name="leg1con_2">
-  <inertial>
-    <origin xyz="-0.02550041106837525 1.1473997643327016e-07 0.006999743573840589" rpy="0 0 0"/>
-    <mass value="0.30660783330227587"/>
-    <inertia ixx="0.000822" iyy="0.000879" izz="7.6e-05" ixy="-0.0" iyz="0.0" ixz="-0.0"/>
-  </inertial>
-  <visual>
-    <origin xyz="0.00668 0.010814 -0.131538" rpy="0 0 0"/>
-    <geometry>
-      <mesh filename="file://$(find tars_robot_description)/meshes/leg1con_2.stl" scale="0.001 0.001 0.001"/>
-    </geometry>
-    <material name="silver"/>
-  </visual>
-  <collision>
-    <origin xyz="0.00668 0.010814 -0.131538" rpy="0 0 0"/>
-    <geometry>
-      <mesh filename="file://$(find tars_robot_description)/meshes/leg1con_2.stl" scale="0.001 0.001 0.001"/>
-    </geometry>
-  </collision>
-</link>
-<link name="leg1con_3">
-  <inertial>
-    <origin xyz="0.025499588931624725 1.1473997643327016e-07 0.00799974357384059" rpy="0 0 0"/>
-    <mass value="0.30660783330227587"/>
-    <inertia ixx="0.000822" iyy="0.000879" izz="7.6e-05" ixy="-0.0" iyz="-0.0" ixz="0.0"/>
-  </inertial>
-  <visual>
-    <origin xyz="-0.02332 0.010814 -0.131538" rpy="0 0 0"/>
-    <geometry>
-      <mesh filename="file://$(find tars_robot_description)/meshes/leg1con_3.stl" scale="0.001 0.001 0.001"/>
-    </geometry>
-    <material name="silver"/>
-  </visual>
-  <collision>
-    <origin xyz="-0.02332 0.010814 -0.131538" rpy="0 0 0"/>
-    <geometry>
-      <mesh filename="file://$(find tars_robot_description)/meshes/leg1con_3.stl" scale="0.001 0.001 0.001"/>
-    </geometry>
-  </collision>
-</link>
-<link name="leg1_1">
-  <inertial>
-    <origin xyz="-0.14250041106837524 1.1473997643500489e-07 0.03899974357384056" rpy="0 0 0"/>
-    <mass value="3.6449999999999996"/>
-    <inertia ixx="0.028431" iyy="0.029046" izz="0.002802" ixy="-0.0" iyz="-0.0" ixz="0.0"/>
-  </inertial>
-  <visual>
-    <origin xyz="-0.04732 0.010814 -0.109538" rpy="0 0 0"/>
-    <geometry>
-      <mesh filename="file://$(find tars_robot_description)/meshes/leg1_1.stl" scale="0.001 0.001 0.001"/>
-    </geometry>
-    <material name="silver"/>
-  </visual>
-  <collision>
-    <origin xyz="-0.04732 0.010814 -0.109538" rpy="0 0 0"/>
-    <geometry>
-      <mesh filename="file://$(find tars_robot_description)/meshes/leg1_1.stl" scale="0.001 0.001 0.001"/>
-    </geometry>
-  </collision>
-</link>
-<link name="leg2_1">
-  <inertial>
-    <origin xyz="0.2744995889316246 1.1473997643673961e-07 0.03799974357384056" rpy="0 0 0"/>
-    <mass value="3.644999999999998"/>
-    <inertia ixx="0.028431" iyy="0.029046" izz="0.002802" ixy="0.0" iyz="-0.0" ixz="-0.0"/>
-  </inertial>
-  <visual>
-    <origin xyz="0.16268 0.010814 -0.111538" rpy="0 0 0"/>
-    <geometry>
-      <mesh filename="file://$(find tars_robot_description)/meshes/leg2_1.stl" scale="0.001 0.001 0.001"/>
-    </geometry>
-    <material name="silver"/>
-  </visual>
-  <collision>
-    <origin xyz="0.16268 0.010814 -0.111538" rpy="0 0 0"/>
-    <geometry>
-      <mesh filename="file://$(find tars_robot_description)/meshes/leg2_1.stl" scale="0.001 0.001 0.001"/>
-    </geometry>
-  </collision>
-</link>
-<joint name="Slider_14" type="prismatic">
-  <origin xyz="-0.00668 -0.010814 0.131538" rpy="0 0 0"/>
-  <parent link="base_link"/>
-  <child link="leg1con_2"/>
-  <axis xyz="0.0 0.0 1.0"/>
-  <limit upper="0.046" lower="0.0" effort="40" velocity="3"/>
-  <dynamics damping="10.0" friction="10.0" />
-</joint>
-<joint name="Slider_15" type="prismatic">
-  <origin xyz="0.02332 -0.010814 0.131538" rpy="0 0 0"/>
-  <parent link="base_link"/>
-  <child link="leg1con_3"/>
-  <axis xyz="0.0 0.0 1.0"/>
-  <limit upper="0.046" lower="0.0" effort="900" velocity="3"/>
-</joint>
-<joint name="Revolute_16" type="revolute">
-  <origin xyz="0.054 0.0 -0.022" rpy="0 0 0"/>
-  <parent link="leg1con_2"/>
-  <child link="leg1_1"/>
-  <axis xyz="1.0 0.0 0.0"/>
-  <limit upper="1.22173" lower="0.0" effort="900" velocity="3"/>
-</joint>
-<joint name="Revolute_17" type="revolute">
-  <origin xyz="-0.186 0.0 -0.02" rpy="0 0 0"/>
-  <parent link="leg1con_3"/>
-  <child link="leg2_1"/>
-  <axis xyz="1.0 0.0 0.0"/>
-  <limit upper="1.22173" lower="0.0" effort="900" velocity="3"/>
-</joint>
-<ros2_control name="GazeboSystem" type="system">
+  </joint>
+  <!-- CENTER BODY (Base Link) -->
+  <link name="base_link">
+    <inertial>
+      <mass value="1.5"/> <!-- center is heavy than the legs  -->
+      <origin xyz="0 0 -0.08" rpy="0 0 0"/> <!-- Center of mass is a littlel bit down so to account for movement -->
+      <inertia ixx="${(1/12)*1.5*(center_height*center_height + center_depth*center_depth)}"
+               iyy="${(1/12)*1.5*(center_height*center_height + center_width*center_width)}"
+               izz="${(1/12)*1.5*(center_width*center_width + center_depth*center_depth)}"
+               ixy="0" ixz="0" iyz="0"/>
+    </inertial>
+    <visual>
+      <origin xyz="0 0 0" rpy="0 0 0"/>
+      <geometry>
+        <box size="${center_depth} ${center_width} ${center_height}"/>
+      </geometry>
+      <material name="silver"/>
+    </visual>
+    <collision>
+      <origin xyz="0 0 0" rpy="0 0 0"/>
+      <geometry>
+        <box size="${center_depth} ${center_width} ${center_height}"/>
+      </geometry>
+    </collision>
+  </link>
+  <!-- This link moves vertically relative to the body (Prismatic Joint) -->
+  <link name="leg_carriage">
+    <inertial>
+      <mass value="0.1"/>
+      <origin xyz="0 0 0" rpy="0 0 0"/>
+      <inertia ixx="0.0001" iyy="0.0001" izz="0.0001" ixy="0" ixz="0" iyz="0"/>
+    </inertial>
+  </link>
+  <joint name="joint_center_linear" type="prismatic">
+    <origin xyz="0 0 -0.0025" rpy="0 0 0"/>
+    <parent link="base_link"/>
+    <child link="leg_carriage"/>
+    <axis xyz="0 0 1"/> <!-- Moves up/down -->
+    <limit lower="-0.046" upper="0.046" effort="100.0" velocity="1.0"/>
+    <dynamics damping="10.0" friction="5.0"/>
+  </joint>
+  <!-- LEFT LEG -->
+  <link name="left_leg">
+    <inertial>
+      <mass value="0.4"/> <!-- legs are lighter than the center body -->
+      <origin xyz="0 0 ${0.04 - leg_height/2 - 0.05}" rpy="0 0 0"/>
+      <inertia ixx="${(1/12)*0.4*(leg_height*leg_height + leg_depth*leg_depth)}"
+               iyy="${(1/12)*0.4*(leg_height*leg_height + leg_width*leg_width)}"
+               izz="${(1/12)*0.4*(leg_width*leg_width + leg_depth*leg_depth)}"
+               ixy="0" ixz="0" iyz="0"/>
+    </inertial>
+    <visual>
+      <origin xyz="0 0 ${0.04 - leg_height/2}" rpy="0 0 0"/>
+      <geometry>
+        <box size="${leg_depth} ${leg_width} ${leg_height}"/>
+      </geometry>
+      <material name="silver"/>
+    </visual>
+    <collision>
+      <origin xyz="0 0 ${0.04 - leg_height/2}" rpy="0 0 0"/>
+      <geometry>
+        <box size="${leg_depth} ${leg_width} ${leg_height}"/>
+      </geometry>
+    </collision>
+  </link>
+  <joint name="joint_left_leg" type="revolute">
+    <origin xyz="0 0.0925 0.09" rpy="0 0 0"/>
+    <parent link="leg_carriage"/>
+    <child link="left_leg"/>
+    <axis xyz="0 1 0"/>
+    <limit lower="-3.14" upper="3.14" effort="100.0" velocity="2.0"/>
+    <dynamics damping="5.0" friction="2.0"/>
+  </joint>
+  <!-- RIGHT LEG -->
+  <link name="right_leg">
+    <inertial>
+      <mass value="0.4"/>   <!-- legs are lighter than the center body -->
+      <origin xyz="0 0 ${0.04 - leg_height/2 - 0.05}" rpy="0 0 0"/>
+      <inertia ixx="${(1/12)*0.4*(leg_height*leg_height + leg_depth*leg_depth)}"
+               iyy="${(1/12)*0.4*(leg_height*leg_height + leg_width*leg_width)}"
+               izz="${(1/12)*0.4*(leg_width*leg_width + leg_depth*leg_depth)}"
+               ixy="0" ixz="0" iyz="0"/>
+    </inertial>
+    <visual>
+      <origin xyz="0 0 ${0.04 - leg_height/2}" rpy="0 0 0"/>
+      <geometry>
+        <box size="${leg_depth} ${leg_width} ${leg_height}"/>
+      </geometry>
+      <material name="silver"/>
+    </visual>
+    <collision>
+      <origin xyz="0 0 ${0.04 - leg_height/2}" rpy="0 0 0"/>
+      <geometry>
+        <box size="${leg_depth} ${leg_width} ${leg_height}"/>
+      </geometry>
+    </collision>
+  </link>
+  <joint name="joint_right_leg" type="revolute">
+    <origin xyz="0 -0.0925 0.09" rpy="0 0 0"/>
+    <parent link="leg_carriage"/>
+    <child link="right_leg"/>
+    <axis xyz="0 1 0"/>
+    <limit lower="-3.14" upper="3.14" effort="100.0" velocity="2.0"/>
+    <dynamics damping="5.0" friction="2.0"/>
+  </joint>
+  <ros2_control name="GazeboSystem" type="system">
     <hardware>
-      <plugin>gazebo_ros2_control/GazeboSystem</plugin>
+      <plugin>ign_ros2_control/IgnitionSystem</plugin>
     </hardware>
-    <joint name="Revolute_16">
+    <joint name="joint_center_linear">
       <command_interface name="position">
-        <param name="min">0</param>
-        <param name="max">1.212198</param>
-      </command_interface>
-      <state_interface name="position"/>
-      <state_interface name="velocity"/>
-    </joint>
-    <joint name="Revolute_17">
-      <command_interface name="position">
-        <param name="min">0</param>
-        <param name="max">1.212198</param>
-      </command_interface>
-      <state_interface name="position"/>
-      <state_interface name="velocity"/>
-    </joint>
-    <joint name="Slider_14">
-      <command_interface name="position">
-        <param name="min">0</param>
+        <param name="min">-0.046</param>
         <param name="max">0.046</param>
       </command_interface>
@@ -161,8 +145,16 @@
       <state_interface name="velocity"/>
     </joint>
-    <joint name="Slider_15">
+    <joint name="joint_left_leg">
       <command_interface name="position">
-        <param name="min">0</param>
-        <param name="max">0.046</param>
+        <param name="min">-3.14</param>
+        <param name="max">3.14</param>
+      </command_interface>
+      <state_interface name="position"/>
+      <state_interface name="velocity"/>
+    </joint>
+    <joint name="joint_right_leg">
+      <command_interface name="position">
+        <param name="min">-3.14</param>
+        <param name="max">3.14</param>
       </command_interface>
       <state_interface name="position"/>
